Commit message: FIX: urdf update filename to current package

File: planning_prm/urdf/scan_pro_robot.urdf.xacro (robot description, xacro)
@@ -18,11 +18,13 @@
 			<origin rpy="0 0 0" xyz="0 0 0"/>
 			<geometry>
-				<mesh filename="package://denso_robot_descriptions/vs6577_description/meshes/base_link.dae" scale="1 1 1"/>
-			</geometry>
-		</visual>
-		<collision>
-			<origin rpy="0 0 0" xyz="0 0 0"/>
-			<geometry>
-				<mesh filename="package://denso_robot_descriptions/vs6577_description/meshes/base_link.dae" scale="1 1 1"/>
+				<!-- <mesh filename="package://denso_robot_descriptions/vs6577_description/meshes/base_link.dae" scale="1 1 1"/> -->
+				<mesh filename="package://planning_prm/meshes/base_link.dae" scale="1 1 1"/>
+			</geometry>
+		</visual>
+		<collision>
+			<origin rpy="0 0 0" xyz="0 0 0"/>
+			<geometry>
+				<!-- <mesh filename="package://denso_robot_descriptions/vs6577_description/meshes/base_link.dae" scale="1 1 1"/> -->
+				<mesh filename="package://planning_prm/meshes/base_link.dae" scale="1 1 1"/>
 			</geometry>
 		</collision>
@@ -37,11 +39,13 @@
 			<origin rpy="0 0 0" xyz="0 0 0"/>
 			<geometry>
-				<mesh filename="package://denso_robot_descriptions/vs6577_description/meshes/J1.dae" scale="1 1 1"/>
-			</geometry>
-		</visual>
-		<collision>
-			<origin rpy="0 0 0" xyz="0 0 0"/>
-			<geometry>
-				<mesh filename="package://denso_robot_descriptions/vs6577_description/meshes/J1.dae" scale="1 1 1"/>
+				<!-- <mesh filename="package://denso_robot_descriptions/vs6577_description/meshes/J1.dae" scale="1 1 1"/> -->
+				<mesh filename="package://planning_prm/meshes/J1.dae" scale="1 1 1"/>
+			</geometry>
+		</visual>
+		<collision>
+			<origin rpy="0 0 0" xyz="0 0 0"/>
+			<geometry>
+				<!-- <mesh filename="package://denso_robot_descriptions/vs6577_description/meshes/J1.dae" scale="1 1 1"/> -->
+				<mesh filename="package://planning_prm/meshes/J1.dae" scale="1 1 1"/>
 			</geometry>
 		</collision>
@@ -56,11 +60,13 @@
 			<origin rpy="0 0 0" xyz="0 0 0"/>
 			<geometry>
-				<mesh filename="package://denso_robot_descriptions/vs6577_description/meshes/J2.dae" scale="1 1 1"/>
-			</geometry>
-		</visual>
-		<collision>
-			<origin rpy="0 0 0" xyz="0 0 0"/>
-			<geometry>
-				<mesh filename="package://denso_robot_descriptions/vs6577_description/meshes/J2.dae" scale="1 1 1"/>
+				<!-- <mesh filename="package://denso_robot_descriptions/vs6577_description/meshes/J2.dae" scale="1 1 1"/> -->
+				<mesh filename="package://planning_prm/meshes/J2.dae" scale="1 1 1"/>
+			</geometry>
+		</visual>
+		<collision>
+			<origin rpy="0 0 0" xyz="0 0 0"/>
+			<geometry>
+				<!-- <mesh filename="package://denso_robot_descriptions/vs6577_description/meshes/J2.dae" scale="1 1 1"/> -->
+				<mesh filename="package://planning_prm/meshes/J2.dae" scale="1 1 1"/>
 			</geometry>
 		</collision>
@@ -75,11 +81,13 @@
 			<origin rpy="0 0 0" xyz="0 0 0"/>
 			<geometry>
-				<mesh filename="package://denso_robot_descriptions/vs6577_description/meshes/J3.dae" scale="1 1 1"/>
-			</geometry>
-		</visual>
-		<collision>
-			<origin rpy="0 0 0" xyz="0 0 0"/>
-			<geometry>
-				<mesh filename="package://denso_robot_descriptions/vs6577_description/meshes/J3.dae" scale="1 1 1"/>
+				<!-- <mesh filename="package://denso_robot_descriptions/vs6577_description/meshes/J3.dae" scale="1 1 1"/> -->
+				<mesh filename="package://planning_prm/meshes/J3.dae" scale="1 1 1"/>
+			</geometry>
+		</visual>
+		<collision>
+			<origin rpy="0 0 0" xyz="0 0 0"/>
+			<geometry>
+				<!-- <mesh filename="package://denso_robot_descriptions/vs6577_description/meshes/J3.dae" scale="1 1 1"/> -->
+				<mesh filename="package://planning_prm/meshes/J3.dae" scale="1 1 1"/>
 			</geometry>
 		</collision>
@@ -94,11 +102,13 @@
 			<origin rpy="0 0 0" xyz="0 0 0"/>
 			<geometry>
-				<mesh filename="package://denso_robot_descriptions/vs6577_description/meshes/J4.dae" scale="1 1 1"/>
-			</geometry>
-		</visual>
-		<collision>
-			<origin rpy="0 0 0" xyz="0 0 0"/>
-			<geometry>
-				<mesh filename="package://denso_robot_descriptions/vs6577_description/meshes/J4.dae" scale="1 1 1"/>
+				<!-- <mesh filename="package://denso_robot_descriptions/vs6577_description/meshes/J4.dae" scale="1 1 1"/> -->
+				<mesh filename="package://planning_prm/meshes/J4.dae" scale="1 1 1"/>
+			</geometry>
+		</visual>
+		<collision>
+			<origin rpy="0 0 0" xyz="0 0 0"/>
+			<geometry>
+				<!-- <mesh filename="package://denso_robot_descriptions/vs6577_description/meshes/J4.dae" scale="1 1 1"/> -->
+				<mesh filename="package://planning_prm/meshes/J4.dae" scale="1 1 1"/>
 			</geometry>
 		</collision>
@@ -113,11 +123,13 @@
 			<origin rpy="0 0 0" xyz="0 0 0"/>
 			<geometry>
-				<mesh filename="package://denso_robot_descriptions/vs6577_description/meshes/J5.dae" scale="1 1 1"/>
-			</geometry>
-		</visual>
-		<collision>
-			<origin rpy="0 0 0" xyz="0 0 0"/>
-			<geometry>
-				<mesh filename="package://denso_robot_descriptions/vs6577_description/meshes/J5.dae" scale="1 1 1"/>
+				<!-- <mesh filename="package://denso_robot_descriptions/vs6577_description/meshes/J5.dae" scale="1 1 1"/> -->
+				<mesh filename="package://planning_prm/meshes/J5.dae" scale="1 1 1"/>
+			</geometry>
+		</visual>
+		<collision>
+			<origin rpy="0 0 0" xyz="0 0 0"/>
+			<geometry>
+				<!-- <mesh filename="package://denso_robot_descriptions/vs6577_description/meshes/J5.dae" scale="1 1 1"/> -->
+				<mesh filename="package://planning_prm/meshes/J5.dae" scale="1 1 1"/>
 			</geometry>
 		</collision>
@@ -132,11 +144,13 @@
 			<origin rpy="0 0 0" xyz="0 0 0"/>
 			<geometry>
-				<mesh filename="package://denso_robot_descriptions/vs6577_description/meshes/J6.dae" scale="1 1 1"/>
-			</geometry>
-		</visual>
-		<collision>
-			<origin rpy="0 0 0" xyz="0 0 0"/>
-			<geometry>
-				<mesh filename="package://denso_robot_descriptions/vs6577_description/meshes/J6.dae" scale="1 1 1"/>
+				<!-- <mesh filename="package://denso_robot_descriptions/vs6577_description/meshes/J6.dae" scale="1 1 1"/> -->
+				<mesh filename="package://planning_prm/meshes/J6.dae" scale="1 1 1"/>
+			</geometry>
+		</visual>
+		<collision>
+			<origin rpy="0 0 0" xyz="0 0 0"/>
+			<geometry>
+				<!-- <mesh filename="package://denso_robot_descriptions/vs6577_description/meshes/J6.dae" scale="1 1 1"/> -->
+				<mesh filename="package://planning_prm/meshes/J6.dae" scale="1 1 1"/>
 			</geometry>
 		</collision>

Commit message: Added transmissions

File: planning_prm/urdf/scan_pro_robot.urdf.xacro (robot description, xacro)
@@ -4,6 +4,7 @@
 	<gazebo>
         <plugin name="gazebo_ros_control" filename="libgazebo_ros_control.so">
-            <robotNamespace>/vs6577</robotNamespace>
-			<legacyModeNS>true</legacyModeNS>
+            <robotNamespace>/</robotNamespace>
+			<controlPeriod>0.001</controlPeriod>
+			<legacyModeNS>false</legacyModeNS>
         </plugin>
     </gazebo>
@@ -236,3 +237,63 @@
 		<dynamics damping="0" friction="0"/>
 	</joint>
+		<transmission name="trans_1">
+		<type>transmission_interface/SimpleTransmission</type>
+		<joint name="joint_1">
+			<hardwareInterface>hardware_interface/PositionJointInterface</hardwareInterface>
+		</joint>
+		<actuator name="motor_1">
+			<hardwareInterface>hardware_interface/PositionJointInterface</hardwareInterface>
+			<mechanicalReduction>1</mechanicalReduction>
+		</actuator>
+	</transmission>
+	<transmission name="trans_2">
+		<type>transmission_interface/SimpleTransmission</type>
+		<joint name="joint_2">
+			<hardwareInterface>hardware_interface/PositionJointInterface</hardwareInterface>
+		</joint>
+		<actuator name="motor_2">
+			<hardwareInterface>hardware_interface/PositionJointInterface</hardwareInterface>
+			<mechanicalReduction>1</mechanicalReduction>
+		</actuator>
+	</transmission>
+	<transmission name="trans_3">
+		<type>transmission_interface/SimpleTransmission</type>
+		<joint name="joint_3">
+			<hardwareInterface>hardware_interface/PositionJointInterface</hardwareInterface>
+		</joint>
+		<actuator name="motor_3">
+			<hardwareInterface>hardware_interface/PositionJointInterface</hardwareInterface>
+			<mechanicalReduction>1</mechanicalReduction>
+		</actuator>
+	</transmission>
+	<transmission name="trans_4">
+		<type>transmission_interface/SimpleTransmission</type>
+		<joint name="joint_4">
+			<hardwareInterface>hardware_interface/PositionJointInterface</hardwareInterface>
+		</joint>
+		<actuator name="motor_4">
+			<hardwareInterface>hardware_interface/PositionJointInterface</hardwareInterface>
+			<mechanicalReduction>1</mechanicalReduction>
+		</actuator>
+	</transmission>
+	<transmission name="trans_5">
+		<type>transmission_interface/SimpleTransmission</type>
+		<joint name="joint_5">
+			<hardwareInterface>hardware_interface/PositionJointInterface</hardwareInterface>
+		</joint>
+		<actuator name="motor_5">
+			<hardwareInterface>hardware_interface/PositionJointInterface</hardwareInterface>
+			<mechanicalReduction>1</mechanicalReduction>
+		</actuator>
+	</transmission>
+	<transmission name="trans_6">
+		<type>transmission_interface/SimpleTransmission</type>
+		<joint name="joint_6">
+			<hardwareInterface>hardware_interface/PositionJointInterface</hardwareInterface>
+		</joint>
+		<actuator name="motor_6">
+			<hardwareInterface>hardware_interface/PositionJointInterface</hardwareInterface>
+			<mechanicalReduction>1</mechanicalReduction>
+		</actuator>
+	</transmission>
 </robot>

Commit message: Added turntable

File: planning_prm/urdf/scan_pro_robot.urdf.xacro (robot description, xacro)
@@ -237,4 +237,70 @@
 		<dynamics damping="0" friction="0"/>
 	</joint>
+    <link name="turntable_base">
+        <visual>
+            <origin rpy="0 0 0" xyz="0 0 0" />
+            <geometry>
+                <cylinder length=".32" radius=".02" />
+            </geometry>
+        </visual>
+        <collision>
+            <origin rpy="0 0 0" xyz="0 0 0" />
+            <geometry>
+                <cylinder length=".32" radius=".02" />
+            </geometry>
+        </collision>
+<inertial>
+            <origin rpy="0 0 0" xyz="0 0 0" />
+            <mass value="1" />
+            <inertia ixx="100" ixy="0" ixz="0" iyy="100" iyz="0" izz="100" />
+        </inertial>
+    </link>
+    <link name="turntable_plate">
+        <visual>
+            <origin rpy="0 0 0" xyz="0 0 0" />
+            <geometry>
+                <cylinder length=".01" radius=".15" />
+            </geometry>
+            <material name="Red">
+                <color rgba="1.0 0 0 1.0" />
+            </material>
+        </visual>
+        <collision>
+            <origin rpy="0 0 0" xyz="0 0 0" />
+            <geometry>
+                <cylinder length=".01" radius=".15" />
+            </geometry>
+        </collision>
+<inertial>
+            <origin rpy="0 0 0" xyz="0 0 0" />
+            <mass value="1" />
+            <inertia ixx="100" ixy="0" ixz="0" iyy="100" iyz="0" izz="100" />
+        </inertial>
+    </link>
+    <joint name="turntable_joint" type="fixed">
+        <!-- <parent link="${parent}"/> -->
+        <parent link="world" />
+        <child link="turntable_base" />
+        <origin rpy="0 0 0" xyz="0 -.6 0.16" />
+        <!-- <origin rpy="0 0 0" xyz="0 0 0" /> -->
+    </joint>
+    <joint name="turntable_revolve_joint" type="continuous">
+        <parent link="turntable_base" />
+        <child link="turntable_plate" />
+        <origin rpy="0.000000 0.000000 0.000000" xyz="0.000000 0.000000 .16" />
+        <!-- <limit effort="1000.0" lower="-6.28" upper="6.28" velocity="0.5"/> -->
+        <limit effort="1000.0" velocity="0.5" />
+        <axis xyz="0 0 1" />
+    </joint>
+    <transmission name="trans_turntable_revolve_joint">
+        <type>transmission_interface/SimpleTransmission</type>
+        <joint name="turntable_revolve_joint">
+            <hardwareInterface>hardware_interface/PositionJointInterface</hardwareInterface>
+        </joint>
+        <actuator name="turntable_revolve_joint_motor">
+            <hardwareInterface>hardware_interface/PositionJointInterface</hardwareInterface>
+            <mechanicalReduction>1</mechanicalReduction>
+        </actuator>
+    </transmission>
 		<transmission name="trans_1">
 		<type>transmission_interface/SimpleTransmission</type>
